Commit message: update

File: src/zbot_description/urdf/zbot_base_old.urdf.xacro (robot description, xacro)
@@ -3,26 +3,26 @@
   name="zbot">
   <link
-    name="base_link">
-    <inertial>
-      <origin
-        xyz="0.000969769171030282 -2.51743070833754E-14 0.112038367342421"
-        rpy="0 0 0" />
-      <mass
-        value="16.3990394222604" />
-      <inertia
-        ixx="0.380637346168345"
-        ixy="-0.148651077561082"
-        ixz="-0.000152996884277864"
-        iyy="0.389495977304953"
-        iyz="3.71624735443284E-16"
-        izz="0.616293577235193" />
-    </inertial>
-    <visual>
-      <origin
-        xyz="0 0 0"
-        rpy="0 0 0" />
-      <geometry>
-        <mesh
-          filename="file://$(env HOME)/zbot_ws/install/zbot_description/share/zbot_description/meshes/base_link.STL" />
+    name="chassis_link">
+    <inertial>
+      <origin
+        xyz="4.1242009807263E-13 -1.41053835278626E-13 0.0457150612516181"
+        rpy="0 0 0" />
+      <mass
+        value="2.91418586484034" />
+      <inertia
+        ixx="0.0160414554493788"
+        ixy="-3.80532779283033E-08"
+        ixz="5.2791865716338E-15"
+        iyy="0.0223949877952289"
+        iyz="3.03477371110732E-16"
+        izz="0.0344217543051772" />
+    </inertial>
+    <visual>
+      <origin
+        xyz="0 0 0"
+        rpy="0 0 0" />
+      <geometry>
+        <mesh
+          filename="file://$(env HOME)/zbot_ws/install/zbot_description/share/zbot_description/meshes/chassis_link.STL" />
       </geometry>
       <material
@@ -34,16 +34,15 @@
     <collision>
       <origin
-        xyz="0 0 0"
-        rpy="0 0 0" />
-      <geometry>
-        <mesh
-          filename="file://$(env HOME)/zbot_ws/install/zbot_description/share/zbot_description/meshes/base_link.STL" />
+        xyz="0 0 0.12"
+        rpy="0 0 0" />
+      <geometry>
+        <box size="0.45 0.45 0.3"/>
       </geometry>
     </collision>
   </link>
   <link name="base_footprint"/>
-  <joint name="basefootprint_to_base" type="fixed">
+  <joint name="basefootprint_to_chassis" type="fixed">
     <parent link="base_footprint"/>
-    <child link="base_link"/>
+    <child link="chassis_link"/>
     <origin xyz="0 0 0.06" rpy="0 0 0"/>
   </joint>
@@ -73,14 +72,14 @@
     </inertial>
   </link>
-  <joint name="base_to_top_box" type="fixed">
-    <parent link="base_link"/>
+  <joint name="chassis_to_top_box" type="fixed">
+    <parent link="chassis_link"/>
     <child link="top_box_link"/>
     <origin xyz="0 0 0.26" rpy="0 0 0"/>
   </joint>
   <link
-    name="Rigthwheel_Link">
-    <inertial>
-      <origin
-        xyz="-2.77555756156289E-17 -0.0172531056477295 3.46944695195361E-17"
+    name="Left_wheel_link">
+    <inertial>
+      <origin
+        xyz="1.38777878078145E-16 0.0172531056477295 7.63278329429795E-16"
         rpy="0 0 0" />
       <mass
@@ -88,8 +87,64 @@
       <inertia
         ixx="0.000450352731222891"
-        ixy="2.93305874890802E-19"
-        ixz="7.95950128490977E-22"
+        ixy="8.63588855368215E-21"
+        ixz="-2.55358655482607E-20"
+        iyy="0.000799166716964205"
+        iyz="-1.56617535979576E-20"
+        izz="0.000450352731222891" />
+    </inertial>
+    <visual>
+      <origin
+        xyz="0 0 0"
+        rpy="0 0 0" />
+      <geometry>
+        <mesh
+          filename="file://$(env HOME)/zbot_ws/install/zbot_description/share/zbot_description/meshes/Left_wheel_link.STL" />
+      </geometry>
+      <material
+        name="">
+        <color
+          rgba="0.792156862745098 0.819607843137255 0.933333333333333 1" />
+      </material>
+    </visual>
+    <collision>
+      <origin
+        xyz="0 0 0"
+        rpy="0 0 0" />
+      <geometry>
+        <mesh
+          filename="file://$(env HOME)/zbot_ws/install/zbot_description/share/zbot_description/meshes/Left_wheel_link.STL" />
+      </geometry>
+    </collision>
+  </link>
+  <joint
+    name="Left_wheel_joint"
+    type="continuous">
+    <origin
+      xyz="0 -0.195500000000004 0"
+      rpy="0 0 0" />
+    <parent
+      link="chassis_link" />
+    <child
+      link="Left_wheel_link" />
+    <axis
+      xyz="0 1 0" />
+    <limit
+      effort="24"
+      velocity="9.42" />
+  </joint>
+  <link
+    name="Right_wheel_link">
+    <inertial>
+      <origin
+        xyz="-1.66533453693773E-16 -0.0172531056477289 -4.16333634234434E-17"
+        rpy="0 0 0" />
+      <mass
+        value="0.422964399925245" />
+      <inertia
+        ixx="0.000450352731222891"
+        ixy="2.9978516071709E-19"
+        ixz="1.86430677315541E-20"
         iyy="0.000799166716964206"
-        iyz="-6.96192737487882E-19"
+        iyz="-6.95386833210546E-19"
         izz="0.000450352731222891" />
     </inertial>
@@ -100,5 +155,5 @@
       <geometry>
         <mesh
-          filename="file://$(env HOME)/zbot_ws/install/zbot_description/share/zbot_description/meshes/Rigthwheel_Link.STL" />
+          filename="file://$(env HOME)/zbot_ws/install/zbot_description/share/zbot_description/meshes/Right_wheel_link.STL" />
       </geometry>
       <material
@@ -114,138 +169,85 @@
       <geometry>
         <mesh
-          filename="file://$(env HOME)/zbot_ws/install/zbot_description/share/zbot_description/meshes/Rigthwheel_Link.STL" />
-      </geometry>
-    </collision>
-  </link>
-  <joint
-    name="Rigthwheel_joint"
-    type="continuous">
-    <origin
-      xyz="0 0.195500000000004 0"
-      rpy="0 0 3.14" />
-    <parent
-      link="base_link" />
-    <child
-      link="Rigthwheel_Link" />
+          filename="file://$(env HOME)/zbot_ws/install/zbot_description/share/zbot_description/meshes/Right_wheel_link.STL" />
+      </geometry>
+    </collision>
+  </link>
+  <joint
+    name="Right_wheel_joint"
+    type="continuous">
+    <origin
+      xyz="0 0.195500000000003 0"
+      rpy="0 0 0" />
+    <parent
+      link="chassis_link" />
+    <child
+      link="Right_wheel_link" />
     <axis
       xyz="0 -1 0" />
-  </joint>
-  <link
-    name="Leftwheel_Link">
-    <inertial>
-      <origin
-        xyz="-2.77555756156289E-17 0.0172531056477295 6.93889390390723E-18"
-        rpy="0 0 0" />
-      <mass
-        value="0.422964399925245" />
-      <inertia
-        ixx="0.000450352731222891"
-        ixy="-1.63319545033364E-21"
-        ixz="-1.17067365193491E-20"
-        iyy="0.000799166716964206"
-        iyz="1.71286555130685E-20"
-        izz="0.000450352731222891" />
-    </inertial>
-    <visual>
-      <origin
-        xyz="0 0 0"
-        rpy="0 0 0" />
-      <geometry>
-        <mesh
-          filename="file://$(env HOME)/zbot_ws/install/zbot_description/share/zbot_description/meshes/Leftwheel_Link.STL" />
-      </geometry>
-      <material
-        name="">
-        <color
-          rgba="0.792156862745098 0.819607843137255 0.933333333333333 1" />
-      </material>
-    </visual>
-    <collision>
-      <origin
-        xyz="0 0 0"
-        rpy="0 0 0" />
-      <geometry>
-        <mesh
-          filename="file://$(env HOME)/zbot_ws/install/zbot_description/share/zbot_description/meshes/Leftwheel_Link.STL" />
-      </geometry>
-    </collision>
-  </link>
-  <joint
-    name="Leftwheel_joint"
-    type="continuous">
-    <origin
-      xyz="0 -0.1955 0"
-      rpy="0 0 0" />
-    <parent
-      link="base_link" />
-    <child
-      link="Leftwheel_Link" />
-    <axis
-      xyz="0 1 0" />
     <limit
       effort="24"
-      velocity="0.58875" />
-  </joint>
-  <link
-    name="Holder1_Link">
-    <inertial>
-      <origin
-        xyz="0.0149538369402379 -2.77555756156289E-17 -0.00548508947688804"
-        rpy="0 0 0" />
-      <mass
-        value="0.0807915502778827" />
-      <inertia
-        ixx="2.45834344225308E-05"
-        ixy="1.69021364418985E-20"
-        ixz="3.88786622376317E-06"
-        iyy="2.66654394263947E-05"
-        iyz="-3.31005941315939E-21"
-        izz="4.19580790977868E-05" />
-    </inertial>
-    <visual>
-      <origin
-        xyz="0 0 0"
-        rpy="0 0 0" />
-      <geometry>
-        <mesh
-          filename="file://$(env HOME)/zbot_ws/install/zbot_description/share/zbot_description/meshes/Holder1_Link.STL" />
-      </geometry>
-      <material
-        name="">
-        <color
-          rgba="0.647058823529412 0.619607843137255 0.588235294117647 1" />
-      </material>
-    </visual>
-    <collision>
-      <origin
-        xyz="0 0 0"
-        rpy="0 0 0" />
-      <geometry>
-        <mesh
-          filename="file://$(env HOME)/zbot_ws/install/zbot_description/share/zbot_description/meshes/Holder1_Link.STL" />
-      </geometry>
-    </collision>
-  </link>
-  <joint
-    name="Holder1_joint"
-    type="continuous">
-    <origin
-      xyz="0.13 0.1295 -0.0075"
-      rpy="0 0 0" />
-    <parent
-      link="base_link" />
-    <child
-      link="Holder1_Link" />
-    <axis
-      xyz="0 0 -1" />
-    <limit
-      effort="0"
-      velocity="0" />
-  </joint>
-  <link
-    name="Wheel1_Link">
-    <inertial>
-      <origin
-        xyz="4.64905891561784E-16 -1.38777878078145E-17 8.23126289350995E-16"
+      velocity="9.42" />
+  </joint>
+  <link
+    name="holder1_Link">
+    <inertial>
+      <origin
+        xyz="0.0149538369402379 0 -0.00548508947688803"
+        rpy="0 0 0" />
+      <mass
+        value="0.0110673356545045" />
+      <inertia
+        ixx="3.36759375651107E-06"
+        ixy="1.91654214425208E-21"
+        ixz="5.32584414214133E-07"
+        iyy="3.65279992142393E-06"
+        iyz="-2.64785319973256E-22"
+        izz="5.74768206818997E-06" />
+    </inertial>
+    <visual>
+      <origin
+        xyz="0 0 0"
+        rpy="0 0 0" />
+      <geometry>
+        <mesh
+          filename="file://$(env HOME)/zbot_ws/install/zbot_description/share/zbot_description/meshes/holder1_Link.STL" />
+      </geometry>
+      <material
+        name="">
+        <color
+          rgba="0 0 0 1" />
+      </material>
+    </visual>
+    <collision>
+      <origin
+        xyz="0 0 0"
+        rpy="0 0 0" />
+      <geometry>
+        <mesh
+          filename="file://$(env HOME)/zbot_ws/install/zbot_description/share/zbot_description/meshes/holder1_Link.STL" />
+      </geometry>
+    </collision>
+  </link>
+  <joint
+    name="holder1_joint"
+    type="continuous">
+    <origin
+      xyz="0.13 0.1295 -0.00949999999999611"
+      rpy="0 0 0" />
+    <parent
+      link="chassis_link" />
+    <child
+      link="holder1_Link" />
+    <axis
+      xyz="0 0 1" />
+    <limit
+      effort="0"
+      velocity="0" />
+  </joint>
+  <link
+    name="wheel1_Link">
+    <inertial>
+      <origin
+        xyz="5.55111512312578E-17 0 3.25260651745651E-18"
         rpy="0 0 0" />
       <mass
@@ -253,8 +255,8 @@
       <inertia
         ixx="1.38792446386636E-05"
-        ixy="-6.31654242534127E-22"
+        ixy="-7.67863316734526E-22"
         ixz="-1.59131939955441E-22"
         iyy="2.33141763250642E-05"
-        iyz="2.23754762315135E-22"
+        iyz="2.27558867913594E-22"
         izz="1.38792446386636E-05" />
     </inertial>
@@ -265,99 +267,99 @@
       <geometry>
         <mesh
-          filename="file://$(env HOME)/zbot_ws/install/zbot_description/share/zbot_description/meshes/Wheel1_Link.STL" />
-      </geometry>
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